Commit message: fix some bugs

File: ros_ws/src/pibot_description/urdf/xbot.urdf (robot description, URDF)
Before this commit: robot xbot_description, 2 links, 1 joints
Joints:
- joint laser_link_joint: origin xyz=0 0 0.7 rpy=0 0 0 -> xyz=0 0 0.7 rpy=0 0 3.1416

Commit message: add xbot with LTME-02A model

File: ros_ws/src/pibot_description/urdf/xbot.urdf (robot description, URDF)
Before this commit: robot xbot_description, 2 links, 1 joints
Links:
- link base_link: mass 10.9839484523713 -> 23.785
- link laser_link: mass 0.17934 -> 0.20612; geometry collision mesh filename=package://pibot_description/meshes/xbot/laser_link.STL; visual mesh filename=package://pibot_description/meshes/xbot/laser_link.STL
Joints:
- joint laser_link_joint: origin xyz=0 0 0.7 rpy=0 0 3.1416 -> xyz=0.3842 0 0.09187 rpy=0 0 0
